File: ninja-keyboard.kicad_pcb (KiCad board)
At the start: 2 copper layers, 300 x 115.3 mm, 125 parts, among them J1 USB_C_Receptacle_USB2.0_14P, J2 Conn_01x02, Q1 CJ3401, SW1 backquote, SW10 num9, SW11 num0, SW12 -, SW13 =, SW14 backsapce, SW15 tab, SW16 q, SW17 w, SW18 e, SW19 r, SW2 num1, SW20 t, SW21 y, SW22 u, SW23 i, SW24 o, SW25 p, SW26 [, SW27 ], SW28 \, SW29 cap, SW3 num2, SW30 a, SW31 s, SW32 d, SW33 f, SW34 h, SW35 g, SW36 j, SW37 k, SW38 l, SW39 semicolon, SW4 num3, SW40 apostrophe, SW41 enter, SW42 pgdown, SW43 lshift, SW44 z, SW45 x, SW46 c, SW47 v, SW48 b, SW49 n, SW5 num4, SW50 m, SW51 comma, SW52 period, SW53 /, SW54 rshift, SW55 up, SW56 end, SW57 lctrl, SW58 win, SW59 lalt, SW6 num5, SW60 lfn, SW61 space, SW62 macro, SW63 rfn, SW64 ralt, SW65 rctrl, SW66 left, SW67 down, SW68 right, SW69 pgup, SW7 num6, SW70 home, SW8 num7, SW9 num8, U1 ESP32-S3-WROOM-1, U2 AMS1117-3.3

Commit message: Lay the components on the board, but haven't connect them with traces
Parts:
- removed C1: 10uF, Capacitor_SMD:C_0603_1608Metric
- removed C2: 0.1uF, Capacitor_SMD:C_0603_1608Metric
- added C10: 0.1uF, Capacitor_SMD:C_0603_1608Metric, B.Cu at (332.1, 155.5)
- added C6: 10uF, Capacitor_SMD:C_0603_1608Metric, B.Cu at (318.7, 148.6)
- added C7: 10uF, Capacitor_SMD:C_0603_1608Metric, B.Cu at (324.0, 143.4)
- added C8: 0.1uF, Capacitor_SMD:C_0603_1608Metric, B.Cu at (321.4, 155.9)
- added C9: 0.1uF, Capacitor_SMD:C_0603_1608Metric, B.Cu at (309.2, 155.7)
- added D38: GREEN, LED_SMD:LED_0603_1608Metric, B.Cu at (326.1, 155.5)
- added D39: Red, LED_SMD:LED_0603_1608Metric, B.Cu at (301.9, 155.7)
- added R10: 4.87k, Resistor_SMD:R_0603_1608Metric, B.Cu at (329.1, 155.5)
- added R11: 47.5k, Resistor_SMD:R_0603_1608Metric, B.Cu at (318.2, 155.9)
- added R12: 10k B=3950 0805, Resistor_SMD:R_0805_2012Metric, B.Cu at (367.6, 151.4)
- added R13: 1.5k, Resistor_SMD:R_0603_1608Metric, B.Cu at (303.6, 155.7)
- added R14: 10k, Resistor_SMD:R_0603_1608Metric, B.Cu at (310.8, 155.7)
- added R15: 11k, Resistor_SMD:R_0603_1608Metric, B.Cu at (312.4, 155.7)
- added R16: 10k, Resistor_SMD:R_0603_1608Metric, B.Cu at (332.1, 152.4)
- added R17: 11k, Resistor_SMD:R_0603_1608Metric, B.Cu at (329.1, 152.3)
- added R6: 1.2k, Resistor_SMD:R_0603_1608Metric, B.Cu at (315.8, 154.0)
- added R9: 3k, Resistor_SMD:R_0603_1608Metric, B.Cu at (326.1, 152.2)
- added U3: TP4056-42-ESOP8, Package_SO:SOIC-8-1EP_3.9x4.9mm_P1.27mm_EP2.41x3.3mm_ThermalVias, B.Cu at (320.9, 152.2)
- D37: value LED_Small -> Yellow
- J2: footprint user_added:1x2 pin gap 1.25mm SMD socket -> user_added:PH 1x2 pin gap 2.0mm SMD socket
- Q1: value CJ3401 -> AO3401A
- R1, R2: footprint Capacitor_SMD:C_0603_1608Metric -> Resistor_SMD:R_0603_1608Metric
- R3: value 10K -> 100K
- R8: value 10K -> 1.5K
- U2: value AMS1117-3.3 -> ~; footprint Package_TO_SOT_SMD:SOT-223-3_TabPin2 -> user_added:XL63020-3.3
- moved R8 22.8 mm to (271.8, 143.9), turned to -90 degrees
- moved D37 21.2 mm to (270.2, 143.9), turned to -90 degrees
- moved Q1 20.0 mm to (320.7, 145.9), turned to 180 degrees
- moved C5 16.0 mm to (267.1, 148.3), turned to -90 degrees
- moved D36 14.8 mm to (315.3, 148.4), turned to -90 degrees
- moved R7 14.5 mm to (268.5, 148.4), turned to 90 degrees
- moved R3 13.5 mm to (314.1, 154.0), turned to -90 degrees
- moved U1 9.23 mm to (255.7, 151.1)
- moved C3 9.23 mm to (267.0, 143.9)
- moved C4 9.23 mm to (268.5, 143.9)
- moved R1 9.23 mm to (267.8, 159.9), turned to 0 degrees
- moved R2 9.23 mm to (267.8, 158.4), turned to 0 degrees
- moved J2 8.70 mm to (329.2, 146.0), turned to -90 degrees
- moved U2 8.62 mm to (286.0, 151.1)
- moved F2 7.10 mm to (311.6, 150.9)
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Connections:
- net /VBAT renamed /BAT+
- net Net-(D36-A) renamed /VCC_5V
- U2 pad 1: GND -> Net-(D36-K)
- U2 pad 2: /3V3 -> GND
- U2 pad 3: Net-(D36-K) -> /3V3
Routing:
- net /VCC_5V: track 0.00 -> 5.49 mm
- net /USB_P: track 0.00 -> 2.99 mm
- net /USB_N: track 0.00 -> 2.90 mm
- net Net-(J1-CC1): track 0.00 -> 2.59 mm
- net /VBUS: track 0.00 -> 2.36 mm
- net Net-(J1-CC2): track 0.00 -> 2.34 mm

Commit message: commit before trying to fix stuck kicad
Parts:
- moved R2 0.48 mm to (267.8, 157.9)
- moved R1 0.47 mm to (267.8, 159.4)
Routing:
- net /3V3: track 0.00 -> 52.4 mm, vias 0 -> 2
- net /USB_P: track 2.99 -> 51.8 mm
- net /USB_N: track 2.90 -> 51.7 mm
- net Net-(D36-K): track 0.00 -> 31.5 mm
- net /BAT+: track 0.00 -> 28.8 mm
- net /CHARG_STATE: track 0.00 -> 27.4 mm, vias 0 -> 4
- net /VCC_5V: track 5.49 -> 28.8 mm
- net /VBUS: track 2.36 -> 9.45 mm
- net /CHIP_UP: track 0.00 -> 5.80 mm
- net /BAT_V_ADC: track 0.00 -> 4.58 mm
- net Net-(U3-TEMP): track 0.00 -> 3.63 mm
- net /EXT_V_ADC: track 0.00 -> 3.22 mm
- net Net-(U3-PROG): track 0.00 -> 2.79 mm
- net Net-(U3-~{STDBY}): track 0.00 -> 2.77 mm
- net Net-(U1-GPIO19/U1RTS/ADC2_CH8/CLK_OUT2/USB_D-): track 0.00 -> 2.62 mm
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Other:
- board text added: "Add switch here"
- board text added: "turning switch"

Commit message: use export netlist feature for now
Parts:
- SW14, SW29: footprint PCM_Switch_Keyboard_Hotswap_Kailh:SW_Hotswap_Kailh_MX_1.75u -> user_added:SW_Hotswap_Kailh_MX_1.75u with led
- SW15, SW54: footprint PCM_Switch_Keyboard_Hotswap_Kailh:SW_Hotswap_Kailh_MX_1.50u -> user_added:SW_Hotswap_Kailh_MX_1.50u with led
- SW28, SW57, SW58, SW59, SW64, SW65: footprint PCM_Switch_Keyboard_Hotswap_Kailh:SW_Hotswap_Kailh_MX_1.25u -> user_added:SW_Hotswap_Kailh_MX_1.25u with led
- SW41: footprint PCM_Switch_Keyboard_Hotswap_Kailh:SW_Hotswap_Kailh_MX_2.00u -> user_added:SW_Hotswap_Kailh_MX_2.00u with led
- SW43, SW61, SW62: footprint PCM_Switch_Keyboard_Hotswap_Kailh:SW_Hotswap_Kailh_MX_2.25u -> user_added:SW_Hotswap_Kailh_MX_2.25u with led
- U1: footprint PCM_Espressif:ESP32-S3-WROOM-1U -> PCM_Espressif:ESP32-S3-WROOM-1
Connections:
- J2 pad 3: GND -> (no net)
- J2 pad 4: GND -> (no net)
- Q1 pad 2: /BAT+ -> Net-(D36-K)
- Q1 pad 3: Net-(D36-K) -> /BAT+
- SW1 pad 1: Net-(SW1-Pad1) -> Net-(SW1-3)
- SW1 pad 3: (no net) -> Net-(SW1-3)
- SW1 pad 4: (no net) -> Net-(SW1-3)
- SW1 pad 5: (no net) -> unconnected-(SW1-DIN-Pad5)
- SW1 pad 6: (no net) -> unconnected-(SW1-GND-Pad6)
- SW10 pad 2: Net-(SW10-Pad2) -> Net-(SW10-5)
- SW10 pad 3: (no net) -> unconnected-(SW10-VDD-Pad3)
- SW10 pad 4: (no net) -> unconnected-(SW10-DOUT-Pad4)
- SW10 pad 5: (no net) -> Net-(SW10-5)
- SW10 pad 6: (no net) -> Net-(SW10-5)
- SW11 pad 1: Net-(SW11-Pad1) -> Net-(SW11-3)
- SW11 pad 3: (no net) -> Net-(SW11-3)
- SW11 pad 4: (no net) -> Net-(SW11-3)
- SW11 pad 5: (no net) -> unconnected-(SW11-DIN-Pad5)
- SW11 pad 6: (no net) -> unconnected-(SW11-GND-Pad6)
- SW12 pad 2: Net-(SW12-Pad2) -> Net-(SW12-5)
- SW12 pad 3: (no net) -> unconnected-(SW12-VDD-Pad3)
- SW12 pad 4: (no net) -> unconnected-(SW12-DOUT-Pad4)
- SW12 pad 5: (no net) -> Net-(SW12-5)
- SW12 pad 6: (no net) -> Net-(SW12-5)
- SW13 pad 1: Net-(SW13-Pad1) -> Net-(SW13-3)
- SW13 pad 3: (no net) -> Net-(SW13-3)
- SW13 pad 4: (no net) -> Net-(SW13-3)
- SW13 pad 5: (no net) -> unconnected-(SW13-DIN-Pad5)
- SW13 pad 6: (no net) -> unconnected-(SW13-GND-Pad6)
- SW14 pad 2: Net-(SW14-Pad2) -> Net-(SW14-5)
- SW15 pad 1: Net-(SW1-Pad1) -> Net-(SW1-3)
- SW16 pad 2: Net-(SW16-Pad2) -> Net-(SW16-5)
- SW16 pad 3: (no net) -> unconnected-(SW16-VDD-Pad3)
- SW16 pad 4: (no net) -> unconnected-(SW16-DOUT-Pad4)
- SW16 pad 5: (no net) -> Net-(SW16-5)
- SW16 pad 6: (no net) -> Net-(SW16-5)
- SW17 pad 1: Net-(SW17-Pad1) -> Net-(SW17-3)
- SW17 pad 3: (no net) -> Net-(SW17-3)
- SW17 pad 4: (no net) -> Net-(SW17-3)
- SW17 pad 5: (no net) -> unconnected-(SW17-DIN-Pad5)
- SW17 pad 6: (no net) -> unconnected-(SW17-GND-Pad6)
- SW18 pad 2: Net-(SW18-Pad2) -> Net-(SW18-5)
- SW18 pad 3: (no net) -> unconnected-(SW18-VDD-Pad3)
- SW18 pad 4: (no net) -> unconnected-(SW18-DOUT-Pad4)
- SW18 pad 5: (no net) -> Net-(SW18-5)
- SW18 pad 6: (no net) -> Net-(SW18-5)
- SW19 pad 1: Net-(SW19-Pad1) -> Net-(SW19-3)
- SW19 pad 3: (no net) -> Net-(SW19-3)
- SW19 pad 4: (no net) -> Net-(SW19-3)
- SW19 pad 5: (no net) -> unconnected-(SW19-DIN-Pad5)
- SW19 pad 6: (no net) -> unconnected-(SW19-GND-Pad6)
- SW2 pad 2: Net-(SW16-Pad2) -> Net-(SW16-5)
- SW2 pad 3: (no net) -> unconnected-(SW2-VDD-Pad3)
- SW2 pad 4: (no net) -> unconnected-(SW2-DOUT-Pad4)
- SW2 pad 5: (no net) -> Net-(SW16-5)
- SW2 pad 6: (no net) -> Net-(SW16-5)
- SW20 pad 2: Net-(SW20-Pad2) -> Net-(SW20-5)
- SW20 pad 3: (no net) -> unconnected-(SW20-VDD-Pad3)
- SW20 pad 4: (no net) -> unconnected-(SW20-DOUT-Pad4)
- SW20 pad 5: (no net) -> Net-(SW20-5)
- SW20 pad 6: (no net) -> Net-(SW20-5)
- SW21 pad 1: Net-(SW21-Pad1) -> Net-(SW21-3)
- SW21 pad 3: (no net) -> Net-(SW21-3)
- SW21 pad 4: (no net) -> Net-(SW21-3)
- SW21 pad 5: (no net) -> unconnected-(SW21-DIN-Pad5)
- SW21 pad 6: (no net) -> unconnected-(SW21-GND-Pad6)
- SW22 pad 2: Net-(SW22-Pad2) -> Net-(SW22-5)
- SW22 pad 3: (no net) -> unconnected-(SW22-VDD-Pad3)
- SW22 pad 4: (no net) -> unconnected-(SW22-DOUT-Pad4)
- SW22 pad 5: (no net) -> Net-(SW22-5)
- SW22 pad 6: (no net) -> Net-(SW22-5)
- SW23 pad 1: Net-(SW23-Pad1) -> Net-(SW23-3)
- SW23 pad 3: (no net) -> Net-(SW23-3)
- SW23 pad 4: (no net) -> Net-(SW23-3)
- SW23 pad 5: (no net) -> unconnected-(SW23-DIN-Pad5)
- SW23 pad 6: (no net) -> unconnected-(SW23-GND-Pad6)
- SW24 pad 2: Net-(SW10-Pad2) -> Net-(SW10-5)
- SW24 pad 3: (no net) -> unconnected-(SW24-VDD-Pad3)
- SW24 pad 4: (no net) -> unconnected-(SW24-DOUT-Pad4)
- SW24 pad 5: (no net) -> Net-(SW10-5)
- SW24 pad 6: (no net) -> Net-(SW10-5)
- SW25 pad 1: Net-(SW11-Pad1) -> Net-(SW11-3)
- SW25 pad 3: (no net) -> Net-(SW11-3)
- SW25 pad 4: (no net) -> Net-(SW11-3)
- SW25 pad 5: (no net) -> unconnected-(SW25-DIN-Pad5)
- SW25 pad 6: (no net) -> unconnected-(SW25-GND-Pad6)
- SW26 pad 2: Net-(SW12-Pad2) -> Net-(SW12-5)
- SW26 pad 3: (no net) -> unconnected-(SW26-VDD-Pad3)
- SW26 pad 4: (no net) -> unconnected-(SW26-DOUT-Pad4)
- SW26 pad 5: (no net) -> Net-(SW12-5)
- SW26 pad 6: (no net) -> Net-(SW12-5)
- SW27 pad 1: Net-(SW13-Pad1) -> Net-(SW13-3)
- SW27 pad 3: (no net) -> Net-(SW13-3)
- SW27 pad 4: (no net) -> Net-(SW13-3)
- SW27 pad 5: (no net) -> unconnected-(SW27-DIN-Pad5)
- SW27 pad 6: (no net) -> unconnected-(SW27-GND-Pad6)
- SW28 pad 2: Net-(SW14-Pad2) -> Net-(SW14-5)
- SW29 pad 1: Net-(SW1-Pad1) -> Net-(SW1-3)
- SW3 pad 1: Net-(SW17-Pad1) -> Net-(SW17-3)
- SW3 pad 3: (no net) -> Net-(SW17-3)
- SW3 pad 4: (no net) -> Net-(SW17-3)
- SW3 pad 5: (no net) -> unconnected-(SW3-DIN-Pad5)
- SW3 pad 6: (no net) -> unconnected-(SW3-GND-Pad6)
- SW30 pad 2: Net-(SW16-Pad2) -> Net-(SW16-5)
- SW30 pad 3: (no net) -> unconnected-(SW30-VDD-Pad3)
- SW30 pad 4: (no net) -> unconnected-(SW30-DOUT-Pad4)
- SW30 pad 5: (no net) -> Net-(SW16-5)
- SW30 pad 6: (no net) -> Net-(SW16-5)
- SW31 pad 1: Net-(SW17-Pad1) -> Net-(SW17-3)
- SW31 pad 3: (no net) -> Net-(SW17-3)
- SW31 pad 4: (no net) -> Net-(SW17-3)
- SW31 pad 5: (no net) -> unconnected-(SW31-DIN-Pad5)
- SW31 pad 6: (no net) -> unconnected-(SW31-GND-Pad6)
- SW32 pad 2: Net-(SW18-Pad2) -> Net-(SW18-5)
- SW32 pad 3: (no net) -> unconnected-(SW32-VDD-Pad3)
- SW32 pad 4: (no net) -> unconnected-(SW32-DOUT-Pad4)
- SW32 pad 5: (no net) -> Net-(SW18-5)
- SW32 pad 6: (no net) -> Net-(SW18-5)
- SW33 pad 1: Net-(SW19-Pad1) -> Net-(SW19-3)
- SW33 pad 3: (no net) -> Net-(SW19-3)
- SW33 pad 4: (no net) -> Net-(SW19-3)
- SW33 pad 5: (no net) -> unconnected-(SW33-DIN-Pad5)
- SW33 pad 6: (no net) -> unconnected-(SW33-GND-Pad6)
- SW34 pad 2: Net-(SW20-Pad2) -> Net-(SW20-5)
- SW34 pad 3: (no net) -> unconnected-(SW34-VDD-Pad3)
- SW34 pad 4: (no net) -> unconnected-(SW34-DOUT-Pad4)
- SW34 pad 5: (no net) -> Net-(SW20-5)
- SW34 pad 6: (no net) -> Net-(SW20-5)
- SW35 pad 1: Net-(SW21-Pad1) -> Net-(SW21-3)
- SW35 pad 3: (no net) -> Net-(SW21-3)
- SW35 pad 4: (no net) -> Net-(SW21-3)
- SW35 pad 5: (no net) -> unconnected-(SW35-DIN-Pad5)
- SW35 pad 6: (no net) -> unconnected-(SW35-GND-Pad6)
- SW36 pad 2: Net-(SW22-Pad2) -> Net-(SW22-5)
- SW36 pad 3: (no net) -> unconnected-(SW36-VDD-Pad3)
- SW36 pad 4: (no net) -> unconnected-(SW36-DOUT-Pad4)
- SW36 pad 5: (no net) -> Net-(SW22-5)
- SW36 pad 6: (no net) -> Net-(SW22-5)
- SW37 pad 1: Net-(SW23-Pad1) -> Net-(SW23-3)
- SW37 pad 3: (no net) -> Net-(SW23-3)
- SW37 pad 4: (no net) -> Net-(SW23-3)
- SW37 pad 5: (no net) -> unconnected-(SW37-DIN-Pad5)
- SW37 pad 6: (no net) -> unconnected-(SW37-GND-Pad6)
- SW38 pad 2: Net-(SW10-Pad2) -> Net-(SW10-5)
- SW38 pad 3: (no net) -> unconnected-(SW38-VDD-Pad3)
- SW38 pad 4: (no net) -> unconnected-(SW38-DOUT-Pad4)
- SW38 pad 5: (no net) -> Net-(SW10-5)
- SW38 pad 6: (no net) -> Net-(SW10-5)
- SW39 pad 1: Net-(SW11-Pad1) -> Net-(SW11-3)
- SW39 pad 3: (no net) -> Net-(SW11-3)
- SW39 pad 4: (no net) -> Net-(SW11-3)
- SW39 pad 5: (no net) -> unconnected-(SW39-DIN-Pad5)
- SW39 pad 6: (no net) -> unconnected-(SW39-GND-Pad6)
- SW4 pad 2: Net-(SW18-Pad2) -> Net-(SW18-5)
- SW4 pad 3: (no net) -> unconnected-(SW4-VDD-Pad3)
- SW4 pad 4: (no net) -> unconnected-(SW4-DOUT-Pad4)
- SW4 pad 5: (no net) -> Net-(SW18-5)
- SW4 pad 6: (no net) -> Net-(SW18-5)
- SW40 pad 2: Net-(SW12-Pad2) -> Net-(SW12-5)
- SW40 pad 3: (no net) -> unconnected-(SW40-VDD-Pad3)
- SW40 pad 4: (no net) -> unconnected-(SW40-DOUT-Pad4)
- SW40 pad 5: (no net) -> Net-(SW12-5)
- SW40 pad 6: (no net) -> Net-(SW12-5)
- SW41 pad 1: Net-(SW13-Pad1) -> Net-(SW13-3)
- SW42 pad 2: Net-(SW14-Pad2) -> Net-(SW14-5)
- SW42 pad 3: (no net) -> unconnected-(SW42-VDD-Pad3)
- SW42 pad 4: (no net) -> unconnected-(SW42-DOUT-Pad4)
- SW42 pad 5: (no net) -> Net-(SW14-5)
- SW42 pad 6: (no net) -> Net-(SW14-5)
- SW43 pad 1: Net-(SW1-Pad1) -> Net-(SW1-3)
- SW44 pad 2: Net-(SW16-Pad2) -> Net-(SW16-5)
- SW44 pad 3: (no net) -> unconnected-(SW44-VDD-Pad3)
- SW44 pad 4: (no net) -> unconnected-(SW44-DOUT-Pad4)
- SW44 pad 5: (no net) -> Net-(SW16-5)
- SW44 pad 6: (no net) -> Net-(SW16-5)
- SW45 pad 1: Net-(SW17-Pad1) -> Net-(SW17-3)
- SW45 pad 3: (no net) -> Net-(SW17-3)
- SW45 pad 4: (no net) -> Net-(SW17-3)
- SW45 pad 5: (no net) -> unconnected-(SW45-DIN-Pad5)
- SW45 pad 6: (no net) -> unconnected-(SW45-GND-Pad6)
- SW46 pad 2: Net-(SW18-Pad2) -> Net-(SW18-5)
- SW46 pad 3: (no net) -> unconnected-(SW46-VDD-Pad3)
- SW46 pad 4: (no net) -> unconnected-(SW46-DOUT-Pad4)
- SW46 pad 5: (no net) -> Net-(SW18-5)
- SW46 pad 6: (no net) -> Net-(SW18-5)
- SW47 pad 1: Net-(SW19-Pad1) -> Net-(SW19-3)
- SW47 pad 3: (no net) -> Net-(SW19-3)
- SW47 pad 4: (no net) -> Net-(SW19-3)
- SW47 pad 5: (no net) -> unconnected-(SW47-DIN-Pad5)
- SW47 pad 6: (no net) -> unconnected-(SW47-GND-Pad6)
- SW48 pad 2: Net-(SW20-Pad2) -> Net-(SW20-5)
- SW48 pad 3: (no net) -> unconnected-(SW48-VDD-Pad3)
- SW48 pad 4: (no net) -> unconnected-(SW48-DOUT-Pad4)
- SW48 pad 5: (no net) -> Net-(SW20-5)
- SW48 pad 6: (no net) -> Net-(SW20-5)
- SW49 pad 1: Net-(SW21-Pad1) -> Net-(SW21-3)
- SW49 pad 3: (no net) -> Net-(SW21-3)
- SW49 pad 4: (no net) -> Net-(SW21-3)
- SW49 pad 5: (no net) -> unconnected-(SW49-DIN-Pad5)
- SW49 pad 6: (no net) -> unconnected-(SW49-GND-Pad6)
- SW5 pad 1: Net-(SW19-Pad1) -> Net-(SW19-3)
- SW5 pad 3: (no net) -> Net-(SW19-3)
- SW5 pad 4: (no net) -> Net-(SW19-3)
- SW5 pad 5: (no net) -> unconnected-(SW5-DIN-Pad5)
- SW5 pad 6: (no net) -> unconnected-(SW5-GND-Pad6)
- SW50 pad 2: Net-(SW22-Pad2) -> Net-(SW22-5)
- SW50 pad 3: (no net) -> unconnected-(SW50-VDD-Pad3)
- SW50 pad 4: (no net) -> unconnected-(SW50-DOUT-Pad4)
- SW50 pad 5: (no net) -> Net-(SW22-5)
- SW50 pad 6: (no net) -> Net-(SW22-5)
- SW51 pad 1: Net-(SW23-Pad1) -> Net-(SW23-3)
- SW51 pad 3: (no net) -> Net-(SW23-3)
- SW51 pad 4: (no net) -> Net-(SW23-3)
- SW51 pad 5: (no net) -> unconnected-(SW51-DIN-Pad5)
- SW51 pad 6: (no net) -> unconnected-(SW51-GND-Pad6)
- SW52 pad 2: Net-(SW10-Pad2) -> Net-(SW10-5)
- SW52 pad 3: (no net) -> unconnected-(SW52-VDD-Pad3)
- SW52 pad 4: (no net) -> unconnected-(SW52-DOUT-Pad4)
- SW52 pad 5: (no net) -> Net-(SW10-5)
- SW52 pad 6: (no net) -> Net-(SW10-5)
- SW53 pad 1: Net-(SW11-Pad1) -> Net-(SW11-3)
- SW53 pad 3: (no net) -> Net-(SW11-3)
- SW53 pad 4: (no net) -> Net-(SW11-3)
- SW53 pad 5: (no net) -> unconnected-(SW53-DIN-Pad5)
- SW53 pad 6: (no net) -> unconnected-(SW53-GND-Pad6)
- SW54 pad 2: Net-(SW12-Pad2) -> Net-(SW12-5)
- SW55 pad 1: Net-(SW13-Pad1) -> Net-(SW13-3)
- SW55 pad 3: (no net) -> Net-(SW13-3)
- SW55 pad 4: (no net) -> Net-(SW13-3)
- SW55 pad 5: (no net) -> unconnected-(SW55-DIN-Pad5)
- SW55 pad 6: (no net) -> unconnected-(SW55-GND-Pad6)
- SW56 pad 2: Net-(SW14-Pad2) -> Net-(SW14-5)
- SW56 pad 3: (no net) -> unconnected-(SW56-VDD-Pad3)
- SW56 pad 4: (no net) -> unconnected-(SW56-DOUT-Pad4)
- SW56 pad 5: (no net) -> Net-(SW14-5)
- SW56 pad 6: (no net) -> Net-(SW14-5)
- SW57 pad 1: Net-(SW1-Pad1) -> Net-(SW1-3)
- SW58 pad 2: Net-(SW16-Pad2) -> Net-(SW16-5)
- SW59 pad 1: Net-(SW17-Pad1) -> Net-(SW17-3)
- SW6 pad 2: Net-(SW20-Pad2) -> Net-(SW20-5)
- SW6 pad 3: (no net) -> unconnected-(SW6-VDD-Pad3)
- SW6 pad 4: (no net) -> unconnected-(SW6-DOUT-Pad4)
- SW6 pad 5: (no net) -> Net-(SW20-5)
- SW6 pad 6: (no net) -> Net-(SW20-5)
- SW60 pad 2: Net-(SW18-Pad2) -> Net-(SW18-5)
- SW60 pad 3: (no net) -> unconnected-(SW60-VDD-Pad3)
- SW60 pad 4: (no net) -> unconnected-(SW60-DOUT-Pad4)
- SW60 pad 5: (no net) -> unconnected-(SW60-DIN-Pad5)
- SW60 pad 6: (no net) -> unconnected-(SW60-GND-Pad6)
- SW61 pad 1: Net-(SW19-Pad1) -> Net-(SW19-3)
- SW62 pad 2: Net-(SW20-Pad2) -> Net-(SW20-5)
- SW63 pad 1: Net-(SW21-Pad1) -> Net-(SW21-3)
- SW63 pad 3: (no net) -> unconnected-(SW63-VDD-Pad3)
- SW63 pad 4: (no net) -> unconnected-(SW63-DOUT-Pad4)
- SW63 pad 5: (no net) -> unconnected-(SW63-DIN-Pad5)
- SW63 pad 6: (no net) -> unconnected-(SW63-GND-Pad6)
- SW64 pad 2: Net-(SW22-Pad2) -> Net-(SW22-5)
- SW65 pad 1: Net-(SW23-Pad1) -> Net-(SW23-3)
- SW66 pad 2: Net-(SW10-Pad2) -> Net-(SW10-5)
- SW66 pad 3: (no net) -> unconnected-(SW66-VDD-Pad3)
- SW66 pad 4: (no net) -> unconnected-(SW66-DOUT-Pad4)
- SW66 pad 5: (no net) -> unconnected-(SW66-DIN-Pad5)
- SW66 pad 6: (no net) -> unconnected-(SW66-GND-Pad6)
- SW67 pad 1: Net-(SW11-Pad1) -> Net-(SW11-3)
- SW67 pad 3: (no net) -> unconnected-(SW67-VDD-Pad3)
- SW67 pad 4: (no net) -> unconnected-(SW67-DOUT-Pad4)
- SW67 pad 5: (no net) -> unconnected-(SW67-DIN-Pad5)
- SW67 pad 6: (no net) -> unconnected-(SW67-GND-Pad6)
- SW68 pad 2: Net-(SW12-Pad2) -> Net-(SW12-5)
- SW68 pad 3: (no net) -> unconnected-(SW68-VDD-Pad3)
- SW68 pad 4: (no net) -> unconnected-(SW68-DOUT-Pad4)
- SW68 pad 5: (no net) -> unconnected-(SW68-DIN-Pad5)
- SW68 pad 6: (no net) -> unconnected-(SW68-GND-Pad6)
- SW69 pad 1: Net-(SW13-Pad1) -> Net-(SW13-3)
- SW69 pad 3: (no net) -> unconnected-(SW69-VDD-Pad3)
- SW69 pad 4: (no net) -> unconnected-(SW69-DOUT-Pad4)
- SW69 pad 5: (no net) -> unconnected-(SW69-DIN-Pad5)
- SW69 pad 6: (no net) -> unconnected-(SW69-GND-Pad6)
- SW7 pad 1: Net-(SW21-Pad1) -> Net-(SW21-3)
- SW7 pad 3: (no net) -> Net-(SW21-3)
- SW7 pad 4: (no net) -> Net-(SW21-3)
- SW7 pad 5: (no net) -> unconnected-(SW7-DIN-Pad5)
- SW7 pad 6: (no net) -> unconnected-(SW7-GND-Pad6)
- SW70 pad 2: Net-(SW14-Pad2) -> Net-(SW14-5)
- SW70 pad 3: (no net) -> unconnected-(SW70-VDD-Pad3)
- SW70 pad 4: (no net) -> unconnected-(SW70-DOUT-Pad4)
- SW70 pad 5: (no net) -> unconnected-(SW70-DIN-Pad5)
- SW70 pad 6: (no net) -> unconnected-(SW70-GND-Pad6)
- SW8 pad 2: Net-(SW22-Pad2) -> Net-(SW22-5)
- SW8 pad 3: (no net) -> unconnected-(SW8-VDD-Pad3)
- SW8 pad 4: (no net) -> unconnected-(SW8-DOUT-Pad4)
- SW8 pad 5: (no net) -> Net-(SW22-5)
- SW8 pad 6: (no net) -> Net-(SW22-5)
- SW9 pad 1: Net-(SW23-Pad1) -> Net-(SW23-3)
- SW9 pad 3: (no net) -> Net-(SW23-3)
- SW9 pad 4: (no net) -> Net-(SW23-3)
- SW9 pad 5: (no net) -> unconnected-(SW9-DIN-Pad5)
- SW9 pad 6: (no net) -> unconnected-(SW9-GND-Pad6)
