File: ninja-keyboard-display/ninja-keyboard-display.kicad_pcb (KiCad board)
At the start: 2 copper layers, 88.6 x 17.9 mm, 8 parts, among them J1 Conn_02x04_Counter_Clockwise, Q1 SS8050

Commit message: Fix DRC errors: connect zone fields
Routing:
- net GND: track 5.91 -> 9.63 mm, vias 33 -> 71
